Commit message: Phase 1: Enhanced URDF with physics, comprehensive world, walking demo
Co-authored-by: ansh1113 <200216682+ansh1113@users.noreply.github.com>

File: src/terrain_description/urdf/anymal_simple.urdf.xacro (robot description, xacro)
@@ -4,7 +4,19 @@
   <xacro:property name="body_length" value="0.6"/>
   <xacro:property name="body_width" value="0.4"/>
-  <xacro:property name="body_height" value="0.15"/>
-  <xacro:property name="leg_length" value="0.35"/>
-  <xacro:property name="foot_radius" value="0.03"/>
+  <xacro:property name="body_height" value="0.2"/>
+  <xacro:property name="upper_leg_length" value="0.3"/>
+  <xacro:property name="lower_leg_length" value="0.3"/>
+  <xacro:property name="foot_radius" value="0.035"/>
+  <!-- Physics properties -->
+  <xacro:property name="body_mass" value="35.0"/>
+  <xacro:property name="hip_mass" value="2.5"/>
+  <xacro:property name="upper_leg_mass" value="2.0"/>
+  <xacro:property name="lower_leg_mass" value="1.2"/>
+  <xacro:property name="foot_mass" value="0.15"/>
+  <!-- Friction and damping -->
+  <xacro:property name="joint_damping" value="0.5"/>
+  <xacro:property name="joint_friction" value="0.1"/>
+  <xacro:property name="foot_friction_mu1" value="1.5"/>
+  <xacro:property name="foot_friction_mu2" value="1.5"/>
   <!-- Materials -->
   <material name="body_color">
@@ -14,5 +26,5 @@
     <color rgba="0.2 0.2 0.2 1.0"/>
   </material>
-  <!-- Base link -->
+  <!-- Base link (body) -->
   <link name="base_link">
     <visual>
@@ -26,12 +38,53 @@
         <box size="${body_length} ${body_width} ${body_height}"/>
       </geometry>
+      <surface>
+        <friction>
+          <ode>
+            <mu>0.8</mu>
+            <mu2>0.8</mu2>
+          </ode>
+        </friction>
+      </surface>
     </collision>
     <inertial>
-      <mass value="30.0"/>
-      <inertia ixx="1.0" ixy="0.0" ixz="0.0" iyy="1.0" iyz="0.0" izz="1.0"/>
+      <origin xyz="0 0 0" rpy="0 0 0"/>
+      <mass value="${body_mass}"/>
+      <inertia
+        ixx="${body_mass * (body_width*body_width + body_height*body_height) / 12.0}"
+        ixy="0.0"
+        ixz="0.0"
+        iyy="${body_mass * (body_length*body_length + body_height*body_height) / 12.0}"
+        iyz="0.0"
+        izz="${body_mass * (body_length*body_length + body_width*body_width) / 12.0}"/>
     </inertial>
   </link>
+  <!-- IMU link -->
+  <link name="imu_link">
+    <inertial>
+      <mass value="0.01"/>
+      <inertia ixx="0.0001" ixy="0" ixz="0" iyy="0.0001" iyz="0" izz="0.0001"/>
+    </inertial>
+  </link>
+  <joint name="imu_joint" type="fixed">
+    <parent link="base_link"/>
+    <child link="imu_link"/>
+    <origin xyz="0 0 0" rpy="0 0 0"/>
+  </joint>
+  <!-- IMU sensor plugin -->
+  <gazebo reference="imu_link">
+    <sensor name="imu_sensor" type="imu">
+      <always_on>true</always_on>
+      <update_rate>100</update_rate>
+      <plugin filename="libgazebo_ros_imu_sensor.so" name="imu_plugin">
+        <ros>
+          <namespace>/</namespace>
+          <remapping>~/out:=imu</remapping>
+        </ros>
+        <initial_orientation_as_reference>false</initial_orientation_as_reference>
+      </plugin>
+    </sensor>
+  </gazebo>
   <!-- Leg macro -->
-  <xacro:macro name="leg" params="name x y">
+  <xacro:macro name="leg" params="name x y reflect">
     <!-- Hip joint (HAA - Hip Abduction/Adduction) -->
     <joint name="${name}_haa_joint" type="revolute">
@@ -40,21 +93,25 @@
       <origin xyz="${x} ${y} 0" rpy="0 0 0"/>
       <axis xyz="1 0 0"/>
-      <limit lower="-0.5" upper="0.5" effort="100" velocity="10"/>
+      <limit lower="-0.4" upper="0.4" effort="80" velocity="12"/>
+      <dynamics damping="${joint_damping}" friction="${joint_friction}"/>
     </joint>
     <link name="${name}_hip_link">
       <visual>
-        <geometry>
-          <cylinder radius="0.05" length="0.1"/>
+        <origin xyz="0 ${reflect*0.03} 0" rpy="0 1.5708 0"/>
+        <geometry>
+          <cylinder radius="0.04" length="0.08"/>
         </geometry>
         <material name="leg_color"/>
       </visual>
       <collision>
-        <geometry>
-          <cylinder radius="0.05" length="0.1"/>
+        <origin xyz="0 ${reflect*0.03} 0" rpy="0 1.5708 0"/>
+        <geometry>
+          <cylinder radius="0.04" length="0.08"/>
         </geometry>
       </collision>
       <inertial>
-        <mass value="2.0"/>
-        <inertia ixx="0.1" ixy="0.0" ixz="0.0" iyy="0.1" iyz="0.0" izz="0.1"/>
+        <origin xyz="0 ${reflect*0.03} 0" rpy="0 0 0"/>
+        <mass value="${hip_mass}"/>
+        <inertia ixx="0.002" ixy="0.0" ixz="0.0" iyy="0.002" iyz="0.0" izz="0.001"/>
       </inertial>
     </link>
@@ -63,26 +120,33 @@
       <parent link="${name}_hip_link"/>
       <child link="${name}_upper_leg_link"/>
-      <origin xyz="0 0 -0.05" rpy="0 0 0"/>
+      <origin xyz="0 ${reflect*0.06} 0" rpy="0 0 0"/>
       <axis xyz="0 1 0"/>
-      <limit lower="-1.5" upper="1.5" effort="100" velocity="10"/>
+      <limit lower="-1.8" upper="1.8" effort="80" velocity="12"/>
+      <dynamics damping="${joint_damping}" friction="${joint_friction}"/>
     </joint>
     <link name="${name}_upper_leg_link">
       <visual>
-        <origin xyz="0 0 -${leg_length/2}" rpy="0 0 0"/>
-        <geometry>
-          <cylinder radius="0.03" length="${leg_length}"/>
+        <origin xyz="0 0 -${upper_leg_length/2}" rpy="0 0 0"/>
+        <geometry>
+          <cylinder radius="0.025" length="${upper_leg_length}"/>
         </geometry>
         <material name="leg_color"/>
       </visual>
       <collision>
-        <origin xyz="0 0 -${leg_length/2}" rpy="0 0 0"/>
-        <geometry>
-          <cylinder radius="0.03" length="${leg_length}"/>
+        <origin xyz="0 0 -${upper_leg_length/2}" rpy="0 0 0"/>
+        <geometry>
+          <cylinder radius="0.025" length="${upper_leg_length}"/>
         </geometry>
       </collision>
       <inertial>
-        <origin xyz="0 0 -${leg_length/2}" rpy="0 0 0"/>
-        <mass value="1.5"/>
-        <inertia ixx="0.1" ixy="0.0" ixz="0.0" iyy="0.1" iyz="0.0" izz="0.01"/>
+        <origin xyz="0 0 -${upper_leg_length/2}" rpy="0 0 0"/>
+        <mass value="${upper_leg_mass}"/>
+        <inertia
+          ixx="${upper_leg_mass * (3*0.025*0.025 + upper_leg_length*upper_leg_length) / 12.0}"
+          ixy="0.0"
+          ixz="0.0"
+          iyy="${upper_leg_mass * (3*0.025*0.025 + upper_leg_length*upper_leg_length) / 12.0}"
+          iyz="0.0"
+          izz="${upper_leg_mass * 0.025*0.025 / 2.0}"/>
       </inertial>
     </link>
@@ -91,26 +155,33 @@
       <parent link="${name}_upper_leg_link"/>
       <child link="${name}_lower_leg_link"/>
-      <origin xyz="0 0 -${leg_length}" rpy="0 0 0"/>
+      <origin xyz="0 0 -${upper_leg_length}" rpy="0 0 0"/>
       <axis xyz="0 1 0"/>
-      <limit lower="-2.5" upper="0.5" effort="100" velocity="10"/>
+      <limit lower="-2.7" upper="0.6" effort="80" velocity="12"/>
+      <dynamics damping="${joint_damping}" friction="${joint_friction}"/>
     </joint>
     <link name="${name}_lower_leg_link">
       <visual>
-        <origin xyz="0 0 -${leg_length/2}" rpy="0 0 0"/>
-        <geometry>
-          <cylinder radius="0.02" length="${leg_length}"/>
+        <origin xyz="0 0 -${lower_leg_length/2}" rpy="0 0 0"/>
+        <geometry>
+          <cylinder radius="0.02" length="${lower_leg_length}"/>
         </geometry>
         <material name="leg_color"/>
       </visual>
       <collision>
-        <origin xyz="0 0 -${leg_length/2}" rpy="0 0 0"/>
-        <geometry>
-          <cylinder radius="0.02" length="${leg_length}"/>
+        <origin xyz="0 0 -${lower_leg_length/2}" rpy="0 0 0"/>
+        <geometry>
+          <cylinder radius="0.02" length="${lower_leg_length}"/>
         </geometry>
       </collision>
       <inertial>
-        <origin xyz="0 0 -${leg_length/2}" rpy="0 0 0"/>
-        <mass value="1.0"/>
-        <inertia ixx="0.05" ixy="0.0" ixz="0.0" iyy="0.05" iyz="0.0" izz="0.005"/>
+        <origin xyz="0 0 -${lower_leg_length/2}" rpy="0 0 0"/>
+        <mass value="${lower_leg_mass}"/>
+        <inertia
+          ixx="${lower_leg_mass * (3*0.02*0.02 + lower_leg_length*lower_leg_length) / 12.0}"
+          ixy="0.0"
+          ixz="0.0"
+          iyy="${lower_leg_mass * (3*0.02*0.02 + lower_leg_length*lower_leg_length) / 12.0}"
+          iyz="0.0"
+          izz="${lower_leg_mass * 0.02*0.02 / 2.0}"/>
       </inertial>
     </link>
@@ -127,8 +198,32 @@
           <sphere radius="${foot_radius}"/>
         </geometry>
+        <surface>
+          <friction>
+            <ode>
+              <mu>${foot_friction_mu1}</mu>
+              <mu2>${foot_friction_mu2}</mu2>
+              <slip1>0.0</slip1>
+              <slip2>0.0</slip2>
+            </ode>
+          </friction>
+          <contact>
+            <ode>
+              <kp>1000000.0</kp>
+              <kd>100.0</kd>
+              <max_vel>0.01</max_vel>
+              <min_depth>0.001</min_depth>
+            </ode>
+          </contact>
+        </surface>
       </collision>
       <inertial>
-        <mass value="0.1"/>
-        <inertia ixx="0.001" ixy="0.0" ixz="0.0" iyy="0.001" iyz="0.0" izz="0.001"/>
+        <mass value="${foot_mass}"/>
+        <inertia
+          ixx="${2.0 * foot_mass * foot_radius * foot_radius / 5.0}"
+          ixy="0.0"
+          ixz="0.0"
+          iyy="${2.0 * foot_mass * foot_radius * foot_radius / 5.0}"
+          iyz="0.0"
+          izz="${2.0 * foot_mass * foot_radius * foot_radius / 5.0}"/>
       </inertial>
     </link>
@@ -136,12 +231,22 @@
       <parent link="${name}_lower_leg_link"/>
       <child link="${name}_foot_link"/>
-      <origin xyz="0 0 -${leg_length}" rpy="0 0 0"/>
-    </joint>
+      <origin xyz="0 0 -${lower_leg_length}" rpy="0 0 0"/>
+    </joint>
+    <!-- Gazebo-specific properties for foot -->
+    <gazebo reference="${name}_foot_link">
+      <mu1>${foot_friction_mu1}</mu1>
+      <mu2>${foot_friction_mu2}</mu2>
+      <kp>1000000.0</kp>
+      <kd>100.0</kd>
+      <minDepth>0.001</minDepth>
+      <maxVel>0.01</maxVel>
+      <material>Gazebo/FlatBlack</material>
+    </gazebo>
   </xacro:macro>
   <!-- Create all four legs -->
-  <xacro:leg name="lf" x="${body_length/2}" y="${body_width/2}"/>
-  <xacro:leg name="rf" x="${body_length/2}" y="-${body_width/2}"/>
-  <xacro:leg name="lh" x="-${body_length/2}" y="${body_width/2}"/>
-  <xacro:leg name="rh" x="-${body_length/2}" y="-${body_width/2}"/>
+  <xacro:leg name="lf" x="${body_length/2-0.05}" y="${body_width/2}" reflect="1"/>
+  <xacro:leg name="rf" x="${body_length/2-0.05}" y="-${body_width/2}" reflect="-1"/>
+  <xacro:leg name="lh" x="-${body_length/2+0.05}" y="${body_width/2}" reflect="1"/>
+  <xacro:leg name="rh" x="-${body_length/2+0.05}" y="-${body_width/2}" reflect="-1"/>
   <!-- Camera sensor -->
   <link name="camera_link">
@@ -159,5 +264,5 @@
     <inertial>
       <mass value="0.1"/>
-      <inertia ixx="0.001" ixy="0.0" ixz="0.0" iyy="0.001" iyz="0.0" izz="0.001"/>
+      <inertia ixx="0.0001" ixy="0.0" ixz="0.0" iyy="0.0001" iyz="0.0" izz="0.0001"/>
     </inertial>
   </link>
@@ -165,9 +270,10 @@
     <parent link="base_link"/>
     <child link="camera_link"/>
-    <origin xyz="${body_length/2} 0 ${body_height/2 + 0.05}" rpy="0 0.3 0"/>
+    <origin xyz="${body_length/2+0.02} 0 ${body_height/2 + 0.03}" rpy="0 0.2 0"/>
   </joint>
   <!-- Camera sensor plugin -->
   <gazebo reference="camera_link">
     <sensor type="camera" name="camera">
+      <always_on>true</always_on>
       <update_rate>30.0</update_rate>
       <camera name="head">
@@ -182,12 +288,19 @@
           <far>300</far>
         </clip>
+        <noise>
+          <type>gaussian</type>
+          <mean>0.0</mean>
+          <stddev>0.007</stddev>
+        </noise>
       </camera>
       <plugin name="camera_controller" filename="libgazebo_ros_camera.so">
-        <alwaysOn>true</alwaysOn>
-        <updateRate>0.0</updateRate>
-        <cameraName>camera</cameraName>
-        <imageTopicName>image_raw</imageTopicName>
-        <cameraInfoTopicName>camera_info</cameraInfoTopicName>
-        <frameName>camera_link</frameName>
+        <ros>
+          <namespace>/</namespace>
+          <remapping>~/image_raw:=camera/image_raw</remapping>
+          <remapping>~/camera_info:=camera/camera_info</remapping>
+        </ros>
+        <camera_name>camera</camera_name>
+        <frame_name>camera_link</frame_name>
+        <hack_baseline>0.07</hack_baseline>
       </plugin>
     </sensor>
@@ -197,5 +310,5 @@
     <visual>
       <geometry>
-        <box size="0.03 0.03 0.03"/>
+        <box size="0.03 0.09 0.03"/>
       </geometry>
       <material name="body_color"/>
@@ -203,10 +316,10 @@
     <collision>
       <geometry>
-        <box size="0.03 0.03 0.03"/>
+        <box size="0.03 0.09 0.03"/>
       </geometry>
     </collision>
     <inertial>
-      <mass value="0.05"/>
-      <inertia ixx="0.0005" ixy="0.0" ixz="0.0" iyy="0.0005" iyz="0.0" izz="0.0005"/>
+      <mass value="0.08"/>
+      <inertia ixx="0.0001" ixy="0.0" ixz="0.0" iyy="0.0001" iyz="0.0" izz="0.0001"/>
     </inertial>
   </link>
@@ -214,12 +327,13 @@
     <parent link="base_link"/>
     <child link="camera_depth_link"/>
-    <origin xyz="${body_length/2} 0.03 ${body_height/2 + 0.05}" rpy="0 0.3 0"/>
+    <origin xyz="${body_length/2+0.02} 0 ${body_height/2 + 0.05}" rpy="0 0.2 0"/>
   </joint>
   <!-- Depth camera sensor plugin -->
   <gazebo reference="camera_depth_link">
     <sensor type="depth" name="depth_camera">
-      <update_rate>30.0</update_rate>
+      <always_on>true</always_on>
+      <update_rate>20.0</update_rate>
       <camera name="depth">
-        <horizontal_fov>1.3962634</horizontal_fov>
+        <horizontal_fov>1.047</horizontal_fov>
         <image>
           <width>640</width>
@@ -228,31 +342,26 @@
         </image>
         <clip>
-          <near>0.05</near>
-          <far>10</far>
+          <near>0.1</near>
+          <far>10.0</far>
         </clip>
+        <noise>
+          <type>gaussian</type>
+          <mean>0.0</mean>
+          <stddev>0.01</stddev>
+        </noise>
       </camera>
-      <plugin name="depth_camera_controller" filename="libgazebo_ros_openni_kinect.so">
-        <baseline>0.2</baseline>
-        <alwaysOn>true</alwaysOn>
-        <updateRate>0.0</updateRate>
-        <cameraName>camera</cameraName>
-        <imageTopicName>rgb/image_raw</imageTopicName>
-        <cameraInfoTopicName>rgb/camera_info</cameraInfoTopicName>
-        <depthImageTopicName>depth/image_raw</depthImageTopicName>
-        <depthImageCameraInfoTopicName>depth/camera_info</depthImageCameraInfoTopicName>
-        <pointCloudTopicName>depth/points</pointCloudTopicName>
-        <frameName>camera_depth_optical_frame</frameName>
-        <pointCloudCutoff>0.5</pointCloudCutoff>
-        <pointCloudCutoffMax>3.0</pointCloudCutoffMax>
-        <distortionK1>0</distortionK1>
-        <distortionK2>0</distortionK2>
-        <distortionK3>0</distortionK3>
-        <distortionT1>0</distortionT1>
-        <distortionT2>0</distortionT2>
-        <CxPrime>0</CxPrime>
-        <Cx>0</Cx>
-        <Cy>0</Cy>
-        <focalLength>0</focalLength>
-        <hackBaseline>0</hackBaseline>
+      <plugin name="depth_camera_controller" filename="libgazebo_ros_camera.so">
+        <ros>
+          <namespace>/</namespace>
+          <remapping>~/image_raw:=camera/depth/image_raw</remapping>
+          <remapping>~/camera_info:=camera/depth/camera_info</remapping>
+          <remapping>~/depth/image_raw:=camera/depth/image_raw</remapping>
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